File: Hardware/PCB/FastStepper.kicad_pcb (KiCad board)
At the start: 4 copper layers, 58 x 77.6 mm, 96 parts, among them IC1 FT232RL, IC10 THS4281DBVT, IC11 M74VHC1GT126DT1G, IC12 M74VHC1GT126DT1G, IC13 M74VHC1GT126DT1G, IC14 M74VHC1GT126DT1G, IC15 M74VHC1GT126DT1G, IC16 M74VHC1GT126DT1G, IC17 M74VHC1GT126DT1G, IC18 M74VHC1GT126DT1G, IC2 M74VHC1GT126DT1G, IC3 LP5907MFX-3.3, IC4 M74VHC1GT126DT1G, IC5 M74VHC1GT126DT1G, IC6 M74VHC1GT126DT1G, IC7 USBLC6-2SC6, IC8 ATXMEGA32A4U, IC9 LP5907MFX-3.3, X1 conn 1x5, X10 conn 1x3, X2 conn 1x2, X3 conn 1x2, X4 conn 1x3, X5 conn 1x5, X6 USB conn, X7 DC_JACK, X8 CLCK_JACK, X9 conn 1x5

Commit message: passo intermédio
Parts:
- removed IC12: M74VHC1GT126DT1G, FastStepper PCBLib:TSOP-5
- removed IC7: USBLC6-2SC6, FastStepper PCBLib:SOT23-6L
- removed IC9: LP5907MFX-3.3, FastStepper PCBLib:TSOT23-5
- removed OSC1: OSCILLATOR, FastStepper PCBLib:OSCILLATOR_3.2X2.5
- removed X7: DC_JACK, FastStepper PCBLib:DC_POWER_INPUT_2.1MM
- removed X8: CLCK_JACK, FastStepper PCBLib:35RASMT2BHNTRX
- added C32: 100nF, Capacitor_SMD:C_0402_1005Metric, F.Cu at (163.5, 138.8)
- added C33: 100nF, Capacitor_SMD:C_0402_1005Metric, F.Cu at (166.9, 126.0)
- added C34: 100nF, Capacitor_SMD:C_0402_1005Metric, F.Cu at (130.7, 72.3)
- added C35: 100nF, Capacitor_SMD:C_0402_1005Metric, F.Cu at (164.1, 132.7)
- added C36: 100nF, Capacitor_SMD:C_0402_1005Metric, F.Cu at (174.3, 106.8)
- added C37: 100nF, Capacitor_SMD:C_0402_1005Metric, F.Cu at (167.2, 112.2)
- added D1: ESD9B3, Diode_SMD:D_SOD-923, F.Cu at (180.4, 103.0)
- added D2: ESD9B3, Diode_SMD:D_SOD-923, F.Cu at (177.8, 89.7)
- added D3: ESD9B3, Diode_SMD:D_SOD-923, F.Cu at (174.3, 103.0)
- added D4: PESD5V0L2BT, Package_TO_SOT_SMD:SOT-23, B.Cu at (181.4, 76.4)
- added D5: PESD5V0L2BT, Package_TO_SOT_SMD:SOT-23, B.Cu at (173.4, 73.6)
- added D6: PESD5V0L2BT, Package_TO_SOT_SMD:SOT-23, B.Cu at (173.4, 76.9)
- added FL1: DLW21HN900SQ2L, FastStepper PCBLib:FIL_DLW21HN900SQ2L, F.Cu at (171.5, 76.9)
- added FL2: DLW21HN900SQ2L, FastStepper PCBLib:FIL_DLW21HN900SQ2L, F.Cu at (171.5, 73.6)
- added IC19: M74VHC1GT126DT1G, Package_SO:TSOP-5_1.65x3.05mm_P0.95mm, F.Cu at (167.5, 137.8)
- added IC20: M74VHC1GT126DT1G, Package_SO:TSOP-5_1.65x3.05mm_P0.95mm, F.Cu at (167.5, 133.8)
- added IC21: M74VHC1GT126DT1G, Package_SO:TSOP-5_1.65x3.05mm_P0.95mm, F.Cu at (131.2, 74.9)
- added IC22: M74VHC1GT126DT1G, Package_SO:TSOP-5_1.65x3.05mm_P0.95mm, F.Cu at (167.5, 129.4)
- added J1: USB_C_Receptacle, Connector_USB:USB_C_Receptacle_Molex_105450-0101, F.Cu at (180.3, 76.2)
- added J2: AudioJack3_Ground_SwitchTR, Connector_Audio:Jack_3.5mm_PJ311_Horizontal, F.Cu at (175.6, 116.3)
- added J3: AudioJack3_Ground_SwitchTR, Connector_Audio:Jack_3.5mm_PJ311_Horizontal, F.Cu at (174.2, 96.5)
- added JP1: SolderJumper_2_Open, Jumper:SolderJumper-2_P1.3mm_Open_RoundedPad1.0x1.5mm, F.Cu at (131.7, 131.9)
- added JP2: SolderJumper_2_Open, Jumper:SolderJumper-2_P1.3mm_Open_RoundedPad1.0x1.5mm, F.Cu at (131.7, 137.3)
- added JP3: SolderJumper_2_Open, Jumper:SolderJumper-2_P1.3mm_Open_RoundedPad1.0x1.5mm, F.Cu at (130.6, 121.5)
- added Q1: AO3401A, Package_TO_SOT_SMD:TSOT-23, F.Cu at (172.5, 88.8)
- added R15: 0R, Resistor_SMD:R_0402_1005Metric, F.Cu at (170.8, 130.4)
- added R16: 10k, Resistor_SMD:R_0402_1005Metric, F.Cu at (131.2, 119.0)
- added R22: 10k, Resistor_SMD:R_0402_1005Metric, F.Cu at (132.4, 134.9)
- added R23: 10k, Resistor_SMD:R_0402_1005Metric, F.Cu at (132.1, 129.3)
- added R24: 1k, Resistor_SMD:R_0402_1005Metric, F.Cu at (159.2, 72.1)
- added R25: 1k, Resistor_SMD:R_0402_1005Metric, F.Cu at (170.8, 109.5)
- added R26: 100k, Resistor_SMD:R_0402_1005Metric, F.Cu at (159.2, 75.9)
- added R27: 100k, Resistor_SMD:R_0402_1005Metric, F.Cu at (159.2, 73.3)
- added U1: 74LVC1G157, Package_SO:TSOP-6_1.65x3.05mm_P0.95mm, F.Cu at (171.3, 106.5)
- added U2: THVD1450D, Package_SO:SOIC-8_3.9x4.9mm_P1.27mm, F.Cu at (165.4, 74.0)
- added U3: ADuM1201BR NOT NORMALLY STOCKED, Package_SO:SOIC-8_3.9x4.9mm_P1.27mm, F.Cu at (164.4, 116.2)
- C1, C12, C13, C14, C16, C17, C18, C19, C2, C20, C21, C22, C25, C26, C27, C28, C29, C3, C30, C31, C4, C41, C42, C5, C6, C7, C9: footprint FastStepper PCBLib:C0402K -> Capacitor_SMD:C_0402_1005Metric
- C10, C11, C15, C8: footprint FastStepper PCBLib:C0603K -> Capacitor_SMD:C_0603_1608Metric
- C23: value 4.7uF -> 100nF; footprint FastStepper PCBLib:C0603K -> Capacitor_SMD:C_0402_1005Metric
- C24: value 4.7uF -> 1u; footprint FastStepper PCBLib:C0603K -> Capacitor_SMD:C_0603_1608Metric
- IC1: footprint FastStepper PCBLib:SSOP28 -> Package_SO:SSOP-28_5.3x10.2mm_P0.65mm
- IC10: footprint FastStepper PCBLib:SOT23-5 -> Package_TO_SOT_SMD:SOT-23-5
- IC11, IC13, IC14, IC15, IC16, IC17, IC18, IC2, IC4, IC5, IC6: footprint FastStepper PCBLib:TSOP-5 -> Package_SO:TSOP-5_1.65x3.05mm_P0.95mm
- IC3: footprint FastStepper PCBLib:TSOT23-5 -> Package_TO_SOT_SMD:TSOT-23-5
- IC8: footprint FastStepper PCBLib:TQFP44 -> Package_QFP:TQFP-44_10x10mm_P0.8mm
- L1, L2, L3: footprint FastStepper PCBLib:R0805 -> Resistor_SMD:R_0805_2012Metric
- R1, R10, R11, R12, R13, R14, R17, R18, R19, R20, R21, R3, R34, R4, R6, R7, R8, R9: footprint FastStepper PCBLib:R0402 -> Resistor_SMD:R_0402_1005Metric
- R2: value 10k -> 100k; footprint FastStepper PCBLib:R0402 -> Resistor_SMD:R_0402_1005Metric
- R5: value 10R -> 1k; footprint FastStepper PCBLib:R0402 -> Resistor_SMD:R_0402_1005Metric
- STATE0: footprint FastStepper PCBLib:CHIP-LED0603 -> LED_SMD:LED_0603_1608Metric
- SV2: footprint FastStepper PCBLib:2X03 -> Connector_PinHeader_2.54mm:PinHeader_2x03_P2.54mm_Vertical
- TP1, TP10, TP13, TP4, TP5, TP6, TP8, TP9: footprint FastStepper PCBLib:TP11R -> TestPoint:TestPoint_THTPad_D1.0mm_Drill0.5mm
- TP11: footprint FastStepper PCBLib:TP11R -> TestPoint:TestPoint_THTPad_D1.0mm_Drill0.5mm; moved to F.Cu
- X1: value conn 1x5 -> conn 1x5 2
- X2: value conn 1x2 -> conn 1x5
- X3: footprint FastStepper PCBLib:22-23-2021 -> FastStepper PCBLib:22-23-2031
- X6: value USB conn -> OSCILLATOR; footprint FastStepper PCBLib:240-0002-1 -> Oscillator:Oscillator_SMD_Abracon_ASE-4Pin_3.2x2.5mm
- moved C24 45.9 mm to (176.0, 106.8), turned to -90 degrees
- moved X1 40.1 mm to (179.9, 133.8)
- moved R2 39.5 mm to (174.3, 104.8), turned to 90 degrees
- moved R5 37.4 mm to (171.6, 103.0), turned to 0 degrees
- moved X6 33.1 mm to (150.6, 92.8), turned to 180 degrees
- moved C3 32.4 mm to (161.5, 112.1), turned to 0 degrees
- moved C23 26.0 mm to (174.9, 80.9)
- moved C2 13.4 mm to (172.6, 81.9), turned to 0 degrees
- moved TP11 5.98 mm to (158.1, 117.1), turned to 0 degrees
- moved C20 4.85 mm to (137.3, 134.4)
- moved IC14 4.85 mm to (136.8, 137.1), turned to 0 degrees
- moved C19 4.80 mm to (137.4, 129.0)
- moved IC13 4.80 mm to (136.8, 131.8), turned to 0 degrees
- moved IC18 4.80 mm to (136.8, 122.6), turned to 0 degrees
- moved R3 4.41 mm to (172.2, 80.3)
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Connections:
- net /USBDM renamed /USB_2u_N
- net /USBDP renamed /USB_2u_P
- C18 pad 1: +3V3 -> GND
- C18 pad 2: GND -> Net-(D2-A2)
- C2 pad 1: Net-(X6-P$3) -> Net-(J1-SHIELD)
- C23 pad 1: +5V -> GND
- C23 pad 2: GND -> Net-(J1-SHIELD)
- C24 pad 1: Net-(IC9-OUT) -> VClk
- C3 pad 1: /USB_POWER -> GND
- C3 pad 2: GND -> VClk
- IC8 pad 12: U_CLOCK_IN -> CLK_2u
- R2 pad 1: U_CLOCK_IN -> VClk
- R2 pad 2: Net-(R2-Pad2) -> Net-(D1-A2)
- R3 pad 2: Net-(X6-P$4) -> Net-(J1-SHIELD)
- R5 pad 1: Net-(IC9-OUT) -> Net-(U1-A)
- R5 pad 2: Net-(R2-Pad2) -> Net-(D3-A2)
- R8 pad 1: EMERGENCY_INPUT -> Net-(IC21-A)
- X1 pad 1: VDD -> +5V
- X1 pad 2: HARP_H2_RX -> /IO stage/2Harp_H2_RX
- X1 pad 3: HARP_H2_TX -> /IO stage/2Harp_H2_TX
- X1 pad 4: HARP_H2_CLOCK_OUT -> /IO stage/2Harp_ClockOut
- X3 pad 1: GND -> unconnected-(X3-Pin_1-Pad1)
- X3 pad 2: EMERGENCY_INPUT -> GND
Routing:
- net U_CLOCK_IN: track 64.0 -> 0.00 mm, vias 3 -> 0
- net CLK_2u: track 0.00 -> 50.9 mm, vias 0 -> 3
- net HARP_H2_TX: track 27.2 -> 5.10 mm
- net HARP_H2_RX: track 26.9 -> 5.88 mm
- net EMERGENCY_INPUT: track 53.9 -> 38.3 mm, vias 1 -> 2
- net VDD: track 14.0 -> 0.00 mm
- net /USB_POWER: track 13.6 -> 0.00 mm, vias 2 -> 0
- net Net-(R2-Pad2): track 13.3 -> 0.00 mm
- net +5V: track 257.3 -> 245.0 mm
- net HARP_H2_CLOCK_OUT: track 9.44 -> 0.00 mm
- net Net-(IC9-OUT): track 8.67 -> 0.00 mm
- net UC_ENDSTOP: track 26.5 -> 17.9 mm
- net +3V3: track 280.0 -> 272.8 mm
- net Net-(IC21-A): track 0.00 -> 6.07 mm, vias 0 -> 2
- net +3.3V_u: track 173.8 -> 168.0 mm
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Other:
- outline, holes or cut-outs redrawn
- board text added: "v.1.?????????????????????????"
- board text removed: "v.1.3 H2"
