File: Hardware/PCB/FastStepper.kicad_pcb (KiCad board)
At the start: 4 copper layers, 61.9 x 84.4 mm, 138 parts, among them IC1 FT232RL, IC10 THS4281DBVT, IC11 M74VHC1GT126DT1G, IC13 M74VHC1GT126DT1G, IC14 M74VHC1GT126DT1G, IC15 M74VHC1GT126DT1G, IC16 M74VHC1GT126DT1G, IC17 M74VHC1GT126DT1G, IC18 M74VHC1GT126DT1G, IC19 M74VHC1GT126DT1G, IC2 M74VHC1GT126DT1G, IC20 M74VHC1GT126DT1G, IC21 M74VHC1GT126DT1G, IC22 M74VHC1GT126DT1G, IC3 LP5907MFX-3.3, IC4 M74VHC1GT126DT1G, IC5 M74VHC1GT126DT1G, IC6 M74VHC1GT126DT1G, IC8 ATXMEGA32A4U, J1 USB_C_Receptacle, J2 PJ-316A-6A, J3 PJ-316A-6A, J4 Keystone 8734, J6 Keystone 8734, Q1 AO3401A, U1 74LVC1G157, U2 THVD1450D, U3 ADUM1201BRZ, X1 conn 1x5 2, X10 conn 1x3, X2 conn 1x5, X3 conn 1x2, X4 conn 1x3, X5 conn 1x5, X6 OSCILLATOR, X9 conn 1x5

Commit message: inicio de redesenho v.1.1
Parts:
- X3: value conn 1x2 -> conn 1x3
Other:
- board text added: "FastStepper v.1.1"
- board text removed: "FastStepper v.1.0"
Changed lines of the file:
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@@
 			)
 		)
-		(property "Value" "conn 1x2"
+		(property "Value" "conn 1x3"
 			(at -3.81 5.08 270)
 			(unlocked yes)
@@
 			)
 		)
-		(property "MPN" "282834-2"
+		(property "MPN" "282834-3"
 			(at 0 0 270)
 			(unlocked yes)
@@
 			)
 		)
-		(property "OEPSPN" "OEPS070020"
+		(property "OEPSPN" "OEPS070035"
 			(at 0 0 270)
 			(unlocked yes)
@@
 		(sheetname "/")
 		(sheetfile "FastStepper.kicad_sch")
-		(attr through_hole exclude_from_pos_files)
+		(attr through_hole exclude_from_pos_files exclude_from_bom dnp)
 		(fp_line
 			(start -0.602448 3.197802)
@@
 		(sheetname "/")
 		(sheetfile "FastStepper.kicad_sch")
-		(attr through_hole exclude_from_pos_files)
+		(attr through_hole exclude_from_pos_files exclude_from_bom dnp)
 		(fp_line
 			(start -0.4 3.4)
@@
 			)
 		)
-		(property "Description" ""
+		(property "Description" "WEIDMUELLER CLAMP CONNECTOR"
 			(at 0 0 90)
 			(layer "F.Fab")
@@
 		)
 	)
-	(gr_text "FastStepper v.1.0"
+	(gr_text "FastStepper v.1.1"
 		(at 143.8 145.3 0)
 		(layer "F.SilkS")
