File: Hardware/PCB/core stage.kicad_sch (KiCad schematic)
At the start: 24 parts, among them IC8 ATXMEGA32A4U

Commit message: passo intermédio
Parts:
- C13, C16, C25, C26, C27, C28, C29: footprint FastStepper PCBLib:C0402K -> Capacitor_SMD:C_0402_1005Metric
- C15: footprint FastStepper PCBLib:C0603K -> Capacitor_SMD:C_0603_1608Metric
- IC8: footprint FastStepper PCBLib:TQFP44 -> Package_QFP:TQFP-44_10x10mm_P0.8mm
- L2, L3: footprint FastStepper PCBLib:R0805 -> Resistor_SMD:R_0805_2012Metric
- R1, R34, R4, R7, R9: footprint FastStepper PCBLib:R0402 -> Resistor_SMD:R_0402_1005Metric
- STATE0: footprint FastStepper PCBLib:CHIP-LED0603 -> LED_SMD:LED_0603_1608Metric
- SV2: footprint FastStepper PCBLib:2X03 -> Connector_PinHeader_2.54mm:PinHeader_2x03_P2.54mm_Vertical
- TP4, TP5, TP6, TP8, TP9: footprint FastStepper PCBLib:TP11R -> TestPoint:TestPoint_THTPad_D1.0mm_Drill0.5mm
- X6: renamed from OSC1; footprint FastStepper PCBLib:OSCILLATOR_3.2X2.5 -> Oscillator:Oscillator_SMD_Abracon_ASE-4Pin_3.2x2.5mm
Connections:
- net +3.3V_u: now also X6.4 (VDD); no longer X6.P$4 (VDD)
- net GND: now also X6.2 (GND); no longer X6.P$2 (GND)
- net at IC8.37 (PR1/XTAL1): now also X6.3 (OUTPUT); no longer X6.P$3 (OUTPUT)
- net U_CLOCK_IN renamed CLK_2u
Other:
- moved on the sheet: L2
