File: Hardware/PCB/core stage.kicad_sch (KiCad schematic)
At the start: 24 parts, among them IC8 ATXMEGA32A4U, X6 OSCILLATOR

Commit message: updated Gerbers & P&P & BOM
Parts:
- C15, R4, R7, R9: now not fitted
Changed lines of the file:
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@@
 		(in_bom yes)
 		(on_board yes)
-		(dnp no)
+		(dnp yes)
 		(fields_autoplaced yes)
 		(property "Reference" "C15"
@@
 		(in_bom yes)
 		(on_board yes)
-		(dnp no)
+		(dnp yes)
 		(fields_autoplaced yes)
 		(property "Reference" "R7"
@@
 		(in_bom yes)
 		(on_board yes)
-		(dnp no)
+		(dnp yes)
 		(fields_autoplaced yes)
 		(property "Reference" "R9"
@@
 		(in_bom yes)
 		(on_board yes)
-		(dnp no)
+		(dnp yes)
 		(fields_autoplaced yes)
 		(property "Reference" "R4"

Commit message: sincronia com v.1.1 de main
Parts:
- C15, R4, R7, R9: OEPSPN n.a. -> OEPS000000
Changed lines of the file:
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@@
 			)
 		)
-		(property "OEPSPN" "n.a."
+		(property "OEPSPN" "OEPS000000"
 			(at 92.71 34.29 0)
 			(effects
@@
 			)
 		)
-		(property "OEPSPN" "n.a."
+		(property "OEPSPN" "OEPS000000"
 			(at 102.87 48.26 0)
 			(effects
@@
 			)
 		)
-		(property "OEPSPN" "n.a."
+		(property "OEPSPN" "OEPS000000"
 			(at 85.09 25.4 90)
 			(effects
@@
 			)
 		)
-		(property "OEPSPN" "n.a."
+		(property "OEPSPN" "OEPS000000"
 			(at 102.87 33.02 0)
 			(effects
